File: logic 7408.v1.1.sch (EAGLE design)
At the start: 5 parts, among them IC1 74HC08D

Commit message: Fixed
Fixed small text error
Other:
- note added: "Logic Block 7408"
- note removed: "Logic Block 4308"
Changed lines of the file:
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@@
 <text x="112.268" y="10.16" size="3.175" layer="94" font="vector" align="bottom-center">More info at
 www.logicblock.me</text>
-<text x="91.44" y="115.57" size="6.4516" layer="94" font="vector" align="center">Logic Block 4308</text>
+<text x="91.44" y="115.57" size="6.4516" layer="94" font="vector" align="center">Logic Block 7408</text>
 <text x="92.71" y="106.68" size="3.81" layer="94" font="vector" align="center">quad 2-input AND gate</text>
 <text x="45.72" y="9.144" size="2.54" layer="94" align="bottom-center">Logic Block project are licenced under Creative
